File: fonte_buck_3V3/fonte_buck_3V3.kicad_sch (KiCad schematic)
At the start: 6 parts, among them U3 LM2594M-3.3

Commit message: changes in stm and add can module
Other:
- title: (none) -> Power Supply 3V3
Changed lines of the file:
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@@
 (kicad_sch (version 20230121) (generator eeschema)
   (paper "A4")
+  (title_block
+    (title "Power Supply 3V3")
+    (date "2023-12-11")
+    (rev "1.0")
+    (comment 1 "Kariston Franzin")
+  )
   (junction (at 146.05 92.075) (diameter 0) (color 0 0 0 0)
   )
@@
     (stroke (width 0) (type default))
   )
-  (polyline (pts (xy 176.53 102.235) (xy 176.53 64.135))
-    (stroke (width 0) (type default))
-  )
   (wire (pts (xy 93.98 81.915) (xy 93.98 78.105))
     (stroke (width 0) (type default))
@@
     (stroke (width 0) (type default))
   )
-  (polyline (pts (xy 81.28 64.135) (xy 176.53 64.135))
-    (stroke (width 0) (type default))
-  )
   (wire (pts (xy 90.17 75.565) (xy 90.17 78.105))
     (stroke (width 0) (type default))
@@
     (stroke (width 0) (type default))
   )
-  (polyline (pts (xy 81.28 64.135) (xy 81.28 102.235))
-    (stroke (width 0) (type default))
-  )
   (wire (pts (xy 119.38 92.075) (xy 119.38 94.615))
     (stroke (width 0) (type default))
@@
   )
   (wire (pts (xy 90.17 78.105) (xy 93.98 78.105))
-    (stroke (width 0) (type default))
-  )
-  (polyline (pts (xy 81.28 102.235) (xy 176.53 102.235))
     (stroke (width 0) (type default))
   )
@@
   )
   (symbol (lib_id "power:+3.3V") (at 162.56 76.835 0) (unit 1)
-    (in_bom yes) (on_board yes) (dnp no)
+    (in_bom yes) (on_board yes) (dnp no) (fields_autoplaced)
     (property "Reference" "#PWR0131" (at 162.56 80.645 0)
       (effects (font (size 1.27 1.27)) hide)
     )
-    (property "Value" "+3.3V" (at 162.941 72.4408 0)
+    (property "Value" "+3.3V" (at 162.56 72.39 0)
       (effects (font (size 1.27 1.27)))
     )
@@
       (project "fonte_buck_3V3"
         (path "/f1acede2-7dfb-41bf-a72d-a0082356905f"
-          (reference "C2") (unit 1)
+          (reference "OUT_C1") (unit 1)
         )
       )
@@
   )
   (symbol (lib_id "power:GND") (at 119.38 94.615 0) (unit 1)
-    (in_bom yes) (on_board yes) (dnp no)
+    (in_bom yes) (on_board yes) (dnp no) (fields_autoplaced)
     (property "Reference" "#PWR0128" (at 119.38 100.965 0)
       (effects (font (size 1.27 1.27)) hide)
     )
-    (property "Value" "GND" (at 119.507 99.0092 0)
+    (property "Value" "GND" (at 119.38 99.06 0)
       (effects (font (size 1.27 1.27)))
     )
@@
       (project "fonte_buck_3V3"
         (path "/f1acede2-7dfb-41bf-a72d-a0082356905f"
-          (reference "L1") (unit 1)
+          (reference "Pwr_L1") (unit 1)
         )
       )
@@
   )
   (symbol (lib_id "power:+12V") (at 90.17 75.565 0) (unit 1)
-    (in_bom yes) (on_board yes) (dnp no)
+    (in_bom yes) (on_board yes) (dnp no) (fields_autoplaced)
     (property "Reference" "#PWR0130" (at 90.17 79.375 0)
       (effects (font (size 1.27 1.27)) hide)
     )
-    (property "Value" "+12V" (at 90.551 71.1708 0)
+    (property "Value" "+12V" (at 90.17 71.12 0)
       (effects (font (size 1.27 1.27)))
     )
@@
   (symbol (lib_id "Device:C") (at 93.98 85.725 0) (unit 1)
     (in_bom yes) (on_board yes) (dnp no) (fields_autoplaced)
-    (property "Reference" "C6" (at 97.79 83.185 0)
-      (effects (font (size 1.27 1.27)) (justify left))
-    )
-    (property "Value" "10uF" (at 97.79 85.725 0)
-      (effects (font (size 1.27 1.27)) (justify left))
+    (property "Reference" "C6" (at 90.17 83.185 0)
+      (effects (font (size 1.27 1.27)) (justify right))
+    )
+    (property "Value" "10uF" (at 90.17 85.725 0)
+      (effects (font (size 1.27 1.27)) (justify right))
     )
     (property "Footprint" "Capacitor_SMD:C_1210_3225Metric" (at 94.9452 89.535 0)
@@
       (effects (font (size 1.27 1.27)) hide)
     )
-    (property "LCSC" "C90143" (at 97.79 88.265 0)
-      (effects (font (size 1.27 1.27)) (justify left))
+    (property "LCSC" "C90143" (at 90.17 88.265 0)
+      (effects (font (size 1.27 1.27)) (justify right))
     )
     (pin "1")
@@
       (project "fonte_buck_3V3"
         (path "/f1acede2-7dfb-41bf-a72d-a0082356905f"
-          (reference "C1") (unit 1)
+          (reference "IN_C1") (unit 1)
         )
       )
@@
       (project "fonte_buck_3V3"
         (path "/f1acede2-7dfb-41bf-a72d-a0082356905f"
-          (reference "U1") (unit 1)
+          (reference "LM2594M1") (unit 1)
         )
       )
@@
       (project "fonte_buck_3V3"
         (path "/f1acede2-7dfb-41bf-a72d-a0082356905f"
-          (reference "C3") (unit 1)
+          (reference "OUT_C2") (unit 1)
         )
       )
@@
       (project "fonte_buck_3V3"
         (path "/f1acede2-7dfb-41bf-a72d-a0082356905f"
-          (reference "D1") (unit 1)
-        )
-      )
-    )
+          (reference "Pwr_D1") (unit 1)
+        )
+      )
+    )
+  )
+  (sheet_instances
+    (path "/" (page "1"))
   )
 )
