File: power_supply_buck_5v/power_supply_buck_5v.kicad_pcb (KiCad board)
At the start: 2 copper layers, 5 parts

Commit message: readme
Routing:
- net GND: track 9.36 -> 9.95 mm, vias 0 -> 45
- added copper zone on F.Cu, net +12V
- added copper zone on B.Cu, net GND
Other:
- board text added: "+12V"
- board text added: "+5V"
- board text added: "GND"
