File: ADS1248/ADS1248/ADS1248.kicad_pcb (KiCad board)
At the start: 2 copper layers, 11 parts

Commit message: add ads1248, RTD multiple sensors 2 wires
Parts:
- added Ads_ain_C1: 0.1uF, Capacitor_SMD:C_0603_1608Metric, F.Cu at (146.9, 97.7)
- added Ads_ain_C2: 0.1uF, Capacitor_SMD:C_0603_1608Metric, F.Cu at (145.4, 99.1)
- added Ads_ain_C3: 0.1uF, Capacitor_SMD:C_0603_1608Metric, F.Cu at (146.9, 100.7)
- added Ads_ain_C4: 0.1uF, Capacitor_SMD:C_0603_1608Metric, F.Cu at (146.9, 91.4)
- added Ads_ain_C5: 0.1uF, Capacitor_SMD:C_0603_1608Metric, F.Cu at (145.4, 92.9)
- added Ads_ain_C6: 0.1uF, Capacitor_SMD:C_0603_1608Metric, F.Cu at (146.9, 94.5)
- added Ads_ref_0_C1: 0.1uF, Capacitor_SMD:C_0603_1608Metric, F.Cu at (146.9, 85.1)
- added Ads_ref_0_C2: 0.1uF, Capacitor_SMD:C_0603_1608Metric, F.Cu at (145.4, 86.7)
- added Ads_ref_0_C3: 0.1uF, Capacitor_SMD:C_0603_1608Metric, F.Cu at (146.9, 88.2)
- added Ads_ref_1_C1: 0.1uF, Capacitor_SMD:C_0603_1608Metric, F.Cu at (181.7, 100.1)
- added Ads_ref_1_C2: 0.1uF, Capacitor_SMD:C_0603_1608Metric, F.Cu at (179.2, 103.5)
- added CRTD_I_CM5: C, Capacitor_SMD:C_0603_1608Metric, F.Cu at (165.0, 91.4)
- added CRTD_I_CM6: C, Capacitor_SMD:C_0603_1608Metric, F.Cu at (165.0, 94.4)
- added CRTD_I_DIFF3: C, Capacitor_SMD:C_0603_1608Metric, F.Cu at (163.5, 93.0)
- added JP_+1: Jumper_2_Open, Jumper:SolderJumper-2_P1.3mm_Open_TrianglePad1.0x1.5mm, F.Cu at (171.4, 89.5)
- added JP_-1: Jumper_2_Open, Jumper:SolderJumper-2_P1.3mm_Open_TrianglePad1.0x1.5mm, F.Cu at (171.4, 92.1)
- added JP_IEXC1: Jumper_2_Open, Jumper:SolderJumper-2_P1.3mm_Open_TrianglePad1.0x1.5mm, F.Cu at (138.7, 88.6)
- added JP_ain0: Jumper_2_Open, Jumper:SolderJumper-2_P1.3mm_Open_TrianglePad1.0x1.5mm, F.Cu at (138.7, 91.3)
- added JP_gnd1: Jumper_2_Open, Jumper:SolderJumper-2_P1.3mm_Open_TrianglePad1.0x1.5mm, F.Cu at (175.8, 103.0)
- added JP_ref_5: Jumper_2_Open, Jumper:SolderJumper-2_P1.3mm_Open_TrianglePad1.0x1.5mm, F.Cu at (175.8, 100.5)
- added JP_ref_refp1: Jumper_2_Open, Jumper:SolderJumper-2_P1.3mm_Open_TrianglePad1.0x1.5mm, F.Cu at (179.1, 100.4)
- added REF1: 10K, Resistor_SMD:R_0603_1608Metric, F.Cu at (143.9, 86.7)
- added Ref_C1: 1uF, Capacitor_SMD:C_0603_1608Metric, F.Cu at (146.2, 77.5)
- added Ref_C2: 22uF, Capacitor_SMD:C_0603_1608Metric, F.Cu at (156.9, 77.7)
- added Ref_C3: 1uF, Capacitor_SMD:C_0603_1608Metric, F.Cu at (155.3, 79.1)
- added U1: REF5050AD, Package_SO:SOIC-8_3.9x4.9mm_P1.27mm, F.Cu at (150.7, 76.4)
- Ads_IC1: footprint Ads1248:SOP65P640X120-28N -> ADS1248:SOP65P640X120-28N
Connections:
- Ads_C2 pad 1: AVDD -> VRefOut
- Ads_C3 pad 1: VRefOut -> AVDD
- Ads_IC1 pad 10: unconnected-(Ads_IC1-VREFCOM-Pad10) -> AVSS
- Ads_IC1 pad 11: unconnected-(Ads_IC1-AIN0/IEXC-Pad11) -> ain0
- Ads_IC1 pad 12: unconnected-(Ads_IC1-AIN1/IEXC-Pad12) -> ain1
- Ads_IC1 pad 13: unconnected-(Ads_IC1-AIN4/IEXC/GPIO4-Pad13) -> ain3
- Ads_IC1 pad 14: unconnected-(Ads_IC1-AIN5/IEXC/GPIO5-Pad14) -> REFP0
- Ads_IC1 pad 15: unconnected-(Ads_IC1-AIN6/IEXC/GPIO6-Pad15) -> ain6
- Ads_IC1 pad 16: unconnected-(Ads_IC1-AIN7/IEXC/GPIO7-Pad16) -> ain7
- Ads_IC1 pad 17: unconnected-(Ads_IC1-AIN2/IEXC/GPIO2-Pad17) -> REFP0
- Ads_IC1 pad 18: unconnected-(Ads_IC1-AIN3/IEXC/GPIO3-Pad18) -> ain3
- Ads_IC1 pad 19: unconnected-(Ads_IC1-IEXC2-Pad19) -> IEXC2
- Ads_IC1 pad 20: unconnected-(Ads_IC1-IEXC1-Pad20) -> IEXC1
- Ads_IC1 pad 5: unconnected-(Ads_IC1-REFP0/GPIO0-Pad5) -> REFP0
- Ads_IC1 pad 6: unconnected-(Ads_IC1-REFN0/GPIO1-Pad6) -> REFN0
- Ads_IC1 pad 7: unconnected-(Ads_IC1-REFP1-Pad7) -> REFP1
- Ads_IC1 pad 8: unconnected-(Ads_IC1-REFN1-Pad8) -> AVSS
Routing:
- net AVSS: track 8.11 -> 13.0 mm
- net AVDD: track 4.99 -> 8.71 mm
- net /5V: track 0.00 -> 2.47 mm
- net Net-(U1-Trim/NR): track 0.00 -> 2.13 mm

Commit message: sinc
Parts:
- moved Ads_ain_C3 29.3 mm to (151.5, 71.8), turned to 0 degrees
- moved Ads_ain_C2 29.2 mm to (150.0, 70.2), turned to 0 degrees
- moved Ads_ain_C1 26.0 mm to (148.5, 71.8), turned to 0 degrees
- moved Ads_ain_C6 25.2 mm to (157.8, 71.8), turned to 0 degrees
- moved Ads_ain_C5 25.1 mm to (156.2, 70.2), turned to 0 degrees
- moved JP_ain0 23.8 mm to (136.8, 67.5), turned to -90 degrees
- moved Ref_C1 22.7 mm to (168.9, 75.8), turned to 0 degrees
- moved Ads_ain_C4 21.2 mm to (154.7, 71.8), turned to 0 degrees
- moved JP_IEXC1 21.1 mm to (139.5, 67.5), turned to -90 degrees
- moved REF1 20.6 mm to (159.7, 73.5), turned to 0 degrees
- moved U1 19.7 mm to (170.0, 80.3), turned to -90 degrees
- moved JP_-1 19.3 mm to (154.3, 101.0), turned to 90 degrees
- moved JP_+1 18.6 mm to (156.9, 101.0), turned to 90 degrees
- moved Ads_ref_0_C2 18.5 mm to (159.7, 75.0), turned to 180 degrees
- moved Ads_ref_1_C1 17.7 mm to (165.4, 107.1), turned to 180 degrees
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Other:
- board outline added: 48 x 58.5 mm
